Commit message: wip: robotiq gripper

File: franka_robotiq_description/urdf/franka_robotiq.urdf.xacro (robot description, xacro)
@@ -1,23 +1,32 @@
 <?xml version="1.0"?>
 <robot name="franka_robotiq" xmlns:xacro="http://www.ros.org/wiki/xacro">
-  <!-- Include the arm -->
+  <xacro:arg name="arm_id" default="panda"/>
+  <xacro:arg name="robot_ip" default=""/>
+  <xacro:arg name="use_fake_hardware" default="false"/>
+  <xacro:arg name="fake_sensor_commands" default="false"/>
+  <xacro:arg name="gripper_com_port" default="/dev/ttyUSB0"/>
+  <!-- Load panda arm -->
   <xacro:include filename="$(find franka_description)/robots/panda_arm.xacro"/>
-  <!-- Include just the Robotiq macro, NOT the full gripper urdf -->
+  <xacro:panda_arm arm_id="$(arg arm_id)" safety_distance="0.03"/>
+  <!-- Load Robotiq Gripper -->
   <xacro:include filename="$(find robotiq_description)/urdf/robotiq_2f_85_macro.urdf.xacro"/>
-  <!-- Instantiate the Franka arm -->
-  <xacro:panda_arm arm_id="panda" safety_distance="0.0"/>
-  <!-- Instantiate the Robotiq gripper once -->
   <xacro:robotiq_gripper
-  name="gripper"
-  prefix=""
-  parent="panda_link8"
-  sim_ignition="false"
-  sim_isaac="false"
-  use_fake_hardware="true"
-  fake_sensor_commands="false"
-  include_ros2_control="true"
-  com_port="/dev/ttyUSB0">
-  <!-- Adjust the gripper mounting pose relative to panda_link8 -->
-  <origin xyz="0 0 -0.03" rpy="0 0 0"/>
-</xacro:robotiq_gripper>
+    name="gripper"
+    prefix=""
+    parent="$(arg arm_id)_link8"
+    sim_ignition="false"
+    sim_isaac="false"
+    use_fake_hardware="$(arg use_fake_hardware)"
+    fake_sensor_commands="$(arg fake_sensor_commands)"
+    include_ros2_control="true"
+    com_port="$(arg gripper_com_port)">
+    <origin xyz="0 0 -0.03" rpy="0 0 0"/>
+  </xacro:robotiq_gripper>
+  <!-- ros2_control for the panda arm -->
+  <xacro:include filename="$(find franka_description)/robots/panda_arm.ros2_control.xacro"/>
+  <xacro:panda_arm_ros2_control
+    ns="$(arg arm_id)"
+    robot_ip="$(arg robot_ip)"
+    use_fake_hardware="$(arg use_fake_hardware)"
+    fake_sensor_commands="$(arg fake_sensor_commands)"/>
 </robot>
